File: Board Files/OpenTendo-AGB.kicad_sch (KiCad schematic)
At the start: 0 parts

Commit message: Add files via upload
Parts:
- added BT1: Battery, OpenTendo-AGB:Battery, symbol Device:Battery
- added C22, C23, C26, C40, C41, C55: 0.1u, OpenTendo-AGB:C_0402_1005Metric, symbol Device:C_Small
- added C24, C57: 1u, OpenTendo-AGB:C_0603_1608Metric, symbol Device:C_Small
- added C25: 0.47u, OpenTendo-AGB:C_0603_1608Metric, symbol Device:C_Small
- added C27, C43: 4.7u, OpenTendo-AGB:C_0805_2012Metric, symbol Device:C_Small
- added C35, C36: 1u, OpenTendo-AGB:C_0805_2012Metric, symbol Device:C_Small
- added C37: 0.01u, OpenTendo-AGB:C_0402_1005Metric, symbol Device:C_Small
- added C44, C56: 2.2u, OpenTendo-AGB:C_0805_2012Metric, symbol Device:C_Small
- added CP1: 100u, OpenTendo-AGB:CP_Elec_5x5.3, symbol Device:C_Polarized_Small
- added CP2: 100u, OpenTendo-AGB:C_Elec_6.3x5.8, symbol Device:C_Polarized_Small
- added CP3: 470u, OpenTendo-AGB:C_Elec_8x10.2, symbol Device:C_Polarized_Small
- added D1: MA112, OpenTendo-AGB:Diode, symbol Device:D
- added D2: RB411D, OpenTendo-AGB:SOT-23, symbol Device:D_Schottky_Dual_Series_KAC_Split
- added D3: RB491D, OpenTendo-AGB:SOT-23, symbol Device:D_Schottky_Dual_Series_KAC_Split
- added DA1, DA2: DA204U, OpenTendo-AGB:SOT-323, symbol Device:D_Dual_Series_AKC_Parallel
- added DL1: SML311UT, OpenTendo-AGB:LED_0603_1608Metric, symbol Device:LED
- added DL2: SML210MT, OpenTendo-AGB:LED_0603_1608Metric, symbol Device:LED
- added F1: 4341.25, OpenTendo-AGB:Fuse_0603_1608Metric, symbol Device:Fuse
- added L1: 100u, OpenTendo-AGB:Inductor, symbol Device:L_Iron
- added Q10: DTC114Y, OpenTendo-AGB:SOT-323, symbol Transistor_BJT:DTC114Y
- added Q4, Q5: FDV303N, OpenTendo-AGB:SOT-23, symbol Transistor_FET:Q_NMOS_SGD
- added Q6: 2SK1582, OpenTendo-AGB:SOT-23, symbol Transistor_FET:Q_NMOS_SGD
- added Q7: SSM3J01F, OpenTendo-AGB:SOT-23, symbol Transistor_FET:Q_PMOS_SGD
- added Q8, Q9: 2SC4081, OpenTendo-AGB:SOT-323, symbol Transistor_BJT:Q_NPN_BEC
- added R10: 470, OpenTendo-AGB:R_0402_1005Metric, symbol Device:R_Small
- added R11, R12, R13: 150, OpenTendo-AGB:R_0402_1005Metric, symbol Device:R_Small
- added R18: 33k, OpenTendo-AGB:R_0402_1005Metric, symbol Device:R_Small
- added R25: 47, OpenTendo-AGB:R_0402_1005Metric, symbol Device:R_Small
- added R26, R34: 15k, OpenTendo-AGB:R_0402_1005Metric, symbol Device:R_Small
- added R32: 1M, OpenTendo-AGB:R_0402_1005Metric, symbol Device:R_Small
- added R33: 5.1, OpenTendo-AGB:R_0402_1005Metric, symbol Device:R_Small
- added SW1: AGB-SW, OpenTendo-AGB:Power Switch, symbol OpenGBA:AGB-SW
- added T1: AGB-XFRM, OpenTendo-AGB:Coil, symbol OpenGBA:AGB-XFRM
- added TP10: VOUT3, OpenTendo-AGB:TestPoint_Pad_D1.0mm_VIA, symbol OpenGBA:TestPoint
- added TP11: VDRV3, OpenTendo-AGB:TestPoint_Pad_D1.0mm, symbol OpenGBA:TestPoint
- added TP113: VDD3, OpenTendo-AGB:TestPoint_Pad_D0.8mm, symbol OpenGBA:TestPoint
- added TP116: T1-6, OpenTendo-AGB:TestPoint_Pad_D1.0mm_VIA, symbol OpenGBA:TestPoint
- added TP12: VDD2, OpenTendo-AGB:TestPoint_Pad_D0.8mm, symbol OpenGBA:TestPoint
- added TP13: VDRV5, OpenTendo-AGB:TestPoint_Pad_D1.0mm, symbol OpenGBA:TestPoint
- added TP14: VOUT5, OpenTendo-AGB:TestPoint_Pad_D0.8mm, symbol OpenGBA:TestPoint
- added TP15: ~{RESET}, OpenTendo-AGB:TestPoint_Pad_D1.25mm_VIA, symbol OpenGBA:TestPoint
- added TP16: D3A, OpenTendo-AGB:TestPoint_Pad_D1.0mm, symbol OpenGBA:TestPoint
- added TP17: D2A, OpenTendo-AGB:TestPoint_Pad_D1.0mm_VIA, symbol OpenGBA:TestPoint
- added TP18: DA2-AC, OpenTendo-AGB:TestPoint_Pad_D0.8mm_VIA, symbol OpenGBA:TestPoint
- added TP19: DA1-AC, OpenTendo-AGB:TestPoint_Pad_D1.0mm_VIA, symbol OpenGBA:TestPoint
- added TP20: DA2-A, OpenTendo-AGB:TestPoint_Pad_D0.8mm, symbol OpenGBA:TestPoint
- added TP21: DA1-C, OpenTendo-AGB:TestPoint_Pad_D0.8mm, symbol OpenGBA:TestPoint
- added TP22: VDD13, OpenTendo-AGB:TestPoint_Pad_D0.8mm, symbol OpenGBA:TestPoint
- added TP23: VDD-15, OpenTendo-AGB:TestPoint_Pad_D1.0mm, symbol OpenGBA:TestPoint
- added TP24: VDD5, OpenTendo-AGB:TestPoint_Pad_D1.0mm, symbol OpenGBA:TestPoint
- added TP25: Q8B, OpenTendo-AGB:TestPoint_Pad_D0.8mm, symbol OpenGBA:TestPoint
- added TP27: Q10B, OpenTendo-AGB:TestPoint_Pad_D0.8mm_VIA, symbol OpenGBA:TestPoint
- added TP28: LOWBAT, OpenTendo-AGB:TestPoint_Pad_D0.8mm, symbol OpenGBA:TestPoint
- added TP29: DL2A, OpenTendo-AGB:TestPoint_Pad_D0.8mm_VIA, symbol OpenGBA:TestPoint
- added TP30: DL2K, OpenTendo-AGB:TestPoint_Pad_D0.8mm_VIA, symbol OpenGBA:TestPoint
- added TP31: DL1A, OpenTendo-AGB:TestPoint_Pad_D0.8mm_VIA, symbol OpenGBA:TestPoint
- added TP32: D1A, OpenTendo-AGB:TestPoint_Pad_D0.8mm_VIA, symbol OpenGBA:TestPoint
- added TP33: Q9C, OpenTendo-AGB:TestPoint_Pad_D1.0mm, symbol OpenGBA:TestPoint
- added TP34: Q9B, OpenTendo-AGB:TestPoint_Pad_D0.8mm, symbol OpenGBA:TestPoint
- added TP83: SW1-2, OpenTendo-AGB:TestPoint_Pad_D1.25mm, symbol OpenGBA:TestPoint
- added TP84: SW1-1, OpenTendo-AGB:TestPoint_Pad_D0.8mm, symbol OpenGBA:TestPoint
- added TP85: VCC, OpenTendo-AGB:TestPoint_Pad_D0.8mm, symbol OpenGBA:TestPoint
- added TP86: C_SCP, OpenTendo-AGB:TestPoint_Pad_D1.0mm, symbol OpenGBA:TestPoint
- added TP87: C_SS5, OpenTendo-AGB:TestPoint_Pad_D1.0mm, symbol OpenGBA:TestPoint
- added TP88: C_SS3, OpenTendo-AGB:TestPoint_Pad_D1.0mm, symbol OpenGBA:TestPoint
- added TP89: VIN, OpenTendo-AGB:TestPoint_Pad_D0.8mm_VIA, symbol OpenGBA:TestPoint
- added TP90: REG_EXT, OpenTendo-AGB:TestPoint_Pad_D0.8mm, symbol OpenGBA:TestPoint
- added TP91: VCNT5, OpenTendo-AGB:TestPoint_Pad_D1.0mm, symbol OpenGBA:TestPoint
- added U10: UMG3N, OpenTendo-AGB:SOT-353_SC-70-5, symbol OpenGBA:UMG3N(4.7K/-)
- added U4: AGB-PMIC, OpenTendo-AGB:TSSOP-16_4.4x5mm_P0.65mm, symbol OpenGBA:AGB-PMIC
Connections:
- new net BT+: BT1.1 (+), F1.1
- new net C_SCP: C25.1, TP86.1, U4.10 (C_SCP)
- new net C_SS3: C22.1, TP88.1, U4.7 (C_SS3)
- new net C_SS5: C23.1, TP87.1, U4.3 (C_SS5)
- new net D1A: D1.2 (A), DL1.1 (K), TP32.1
- new net D2A: D2.2 (A), Q4.3 (D), T1.1, T1.2, TP17.1
- new net D3A: D3.2 (A), L1.2, Q5.3 (D), TP16.1
- new net DA1-AC: C40.1, DA1.3 (common), TP19.1
- new net DA1-C: DA1.2 (K), R11.1, TP21.1
- new net DA2-A: DA2.1 (A), R12.1, TP20.1
- new net DA2-AC: C41.1, DA2.3 (common), TP18.1
- new net DL1A: DL1.2 (A), R25.2, TP31.1
- new net DL2A: DL2.2 (A), R10.2, TP29.1
- new net DL2K: DL2.1 (K), TP30.1, U10.5 (1C)
- new net GND: BT1.2 (-), C22.2, C23.2, C24.2, C25.2, C26.2, C27.2, C35.2, C36.2, C43.2, C44.2, C55.2, C56.2, CP1.2, CP2.2, CP3.2, DA1.1 (A), DA2.2 (K), Q10.2 (E), Q4.1 (S), Q5.1 (S), Q9.2 (E), R13.2, SW1.5 (SH), T1.8, U10.2 (E), U4.5 (GND)
- new net LOWBAT: R18.2, TP28.1, U10.1 (1B), U10.3 (2B), U4.15 (~{LOWBAT})
- new net Q10B: C57.1, Q10.1 (B), TP27.1
- new net Q8B: Q10.3 (C), Q8.1 (B), R34.1, TP25.1
- new net Q9B: Q9.1 (B), R26.2, TP34.1, U10.4 (2C)
- new net Q9C: D1.1 (K), Q9.3 (C), TP33.1
- new net REG_EXT: C37.2, Q7.2 (G), R32.2, TP90.1, U4.11 (REG_EXT)
- new net SW1-1: R13.1, SW1.1, TP84.1
- new net SW1-2: F1.2, SW1.4 (2), TP83.1
- new net T1-6: C40.2, C41.2, T1.6, TP116.1
- new net VCC: C43.1, CP1.1, L1.1, R25.1, R33.1, SW1.2 (C), SW1.3 (C), T1.3, T1.4, TP85.1
- new net VCNT5: TP91.1, U4.9 (VCNT5)
- new net VDD-15: C36.1, R12.2, TP23.1
- new net VDD13: C35.1, Q6.2 (G), Q8.3 (C), R11.2, TP22.1, U4.16 (VS13)
- new net VDD2: C27.1, TP12.1, U4.13 (VS2)
- new net VDD3: C26.1, C44.1, Q7.3 (D), R10.1, R18.1, R26.1, TP113.1, U4.12 (REG_FB)
- new net VDD5: C56.1, Q6.1 (S), Q8.2 (E), TP24.1
- new net VDRV3: Q5.2 (G), TP11.1, U4.6 (VDRV3)
- new net VDRV5: Q4.2 (G), TP13.1, U4.4 (VDRV5)
- new net VIN: C24.1, R33.2, TP89.1, U4.1 (VIN)
- new net VOUT3: C37.1, C55.1, CP3.1, D3.3 (K), Q7.1 (S), R32.1, TP10.1, U4.8 (VOUT3)
- new net VOUT5: CP2.1, D2.3 (K), Q6.3 (D), TP14.1, U4.2 (VOUT5)
- new net VSHD: C57.2, R34.2
- new net ~{RESET}: TP15.1, U4.14 (~{RESET})
- no-connect marks 0 -> 2
Other:
- added sheet CPU (CPU.kicad_sch)
- title: (none) -> OpenTendo-AGB
